Commit message: updated urdf

File: ros2/src/cube_description/urdf/cube.xacro (robot description, xacro)
@@ -5,21 +5,14 @@
 <xacro:include filename="$(find cube_description)/urdf/gazebo.xacro" />
 <link name="base_footprint">
-  <visual>
-    <origin xyz="0 0 0" rpy="0 0 0" />
-    <geometry>
-      <box size="0.0 0.0 0.0" />
-    </geometry>
-  </visual>
 </link>
 <joint name="fixed_base_joint" type="fixed">
   <parent link="base_footprint" />
   <child link="base_link" />
-  <origin xyz="0 0 0" rpy="0 0 0" />
 </joint>
 <link name="base_link">
   <inertial>
-    <origin xyz="1.9410706945315624e-05 7.449572592086158e-17 0.07325173847508996" rpy="0 0 0"/>
-    <mass value="92.00463500203875"/>
-    <inertia ixx="1.293901" iyy="2.461346" izz="3.694097" ixy="-0.0" iyz="0.0" ixz="-4e-06"/>
+    <origin xyz="-0.03436104134763452 0.004255153166517912 0.20134904683591295" rpy="0 0 0"/>
+    <mass value="47.20765989840476"/>
+    <inertia ixx="1.033748" iyy="1.280415" izz="1.201" ixy="0.031639" iyz="-0.040215" ixz="0.114859"/>
   </inertial>
   <visual>
@@ -28,5 +21,5 @@
       <mesh filename="package://cube_description/meshes/base_link.stl" scale="0.001 0.001 0.001"/>
     </geometry>
-    <material name="steel_satin"/>
+    <material name="opaque160160160"/>
   </visual>
   <collision>
@@ -39,17 +32,17 @@
 <link name="imu_v1_1">
   <inertial>
-    <origin xyz="0.0 0.0 0.0050000000000000044" rpy="0 0 0"/>
-    <mass value="0.07064999999999999"/>
-    <inertia ixx="6e-06" iyy="6e-06" izz="1.1e-05" ixy="0.0" iyz="0.0" ixz="0.0"/>
+    <origin xyz="0.01122185649964677 0.007537279025856644 0.0010632487781882527" rpy="0 0 0"/>
+    <mass value="0.007717572133230737"/>
+    <inertia ixx="0.0" iyy="0.0" izz="1e-06" ixy="0.0" iyz="0.0" ixz="-0.0"/>
   </inertial>
   <visual>
-    <origin xyz="0.1 -0.0 -0.1055" rpy="0 0 0"/>
+    <origin xyz="0.052922 0.082837 -0.2515" rpy="0 0 0"/>
     <geometry>
       <mesh filename="package://cube_description/meshes/imu_v1_1.stl" scale="0.001 0.001 0.001"/>
     </geometry>
-    <material name="steel_satin"/>
+    <material name="opaque262626"/>
   </visual>
   <collision>
-    <origin xyz="0.1 -0.0 -0.1055" rpy="0 0 0"/>
+    <origin xyz="0.052922 0.082837 -0.2515" rpy="0 0 0"/>
     <geometry>
       <mesh filename="package://cube_description/meshes/imu_v1_1.stl" scale="0.001 0.001 0.001"/>
@@ -57,12 +50,32 @@
   </collision>
 </link>
+<link name="lidar_v1_1">
+  <inertial>
+    <origin xyz="-0.0006310310009192133 -1.036682722385878e-06 -0.0005403106637103805" rpy="0 0 0"/>
+    <mass value="1.347912159118483"/>
+    <inertia ixx="0.000658" iyy="0.000639" izz="0.000873" ixy="0.0" iyz="0.0" ixz="7e-06"/>
+  </inertial>
+  <visual>
+    <origin xyz="-0.128043 1.5e-05 -0.1955" rpy="0 0 0"/>
+    <geometry>
+      <mesh filename="package://cube_description/meshes/lidar_v1_1.stl" scale="0.001 0.001 0.001"/>
+    </geometry>
+    <material name="steel_satin"/>
+  </visual>
+  <collision>
+    <origin xyz="-0.128043 1.5e-05 -0.1955" rpy="0 0 0"/>
+    <geometry>
+      <mesh filename="package://cube_description/meshes/lidar_v1_1.stl" scale="0.001 0.001 0.001"/>
+    </geometry>
+  </collision>
+</link>
 <link name="depth_camera_v1_1">
   <inertial>
-    <origin xyz="0.006500000000000061 -3.011479954295737e-17 0.0" rpy="0 0 0"/>
-    <mass value="0.06123000182479622"/>
-    <inertia ixx="1.9e-05" iyy="1e-06" izz="1.9e-05" ixy="0.0" iyz="0.0" ixz="0.0"/>
+    <origin xyz="0.012822415314312635 0.02438009637633534 -1.0027264107370648e-05" rpy="0 0 0"/>
+    <mass value="0.4030868295259092"/>
+    <inertia ixx="0.000247" iyy="4.1e-05" izz="0.000247" ixy="6e-06" iyz="-0.0" ixz="-0.0"/>
   </inertial>
   <visual>
-    <origin xyz="-0.28 0.0 -0.0805" rpy="0 0 0"/>
+    <origin xyz="-0.184088 0.022403 -0.1615" rpy="0 0 0"/>
     <geometry>
       <mesh filename="package://cube_description/meshes/depth_camera_v1_1.stl" scale="0.001 0.001 0.001"/>
@@ -71,5 +84,5 @@
   </visual>
   <collision>
-    <origin xyz="-0.28 0.0 -0.0805" rpy="0 0 0"/>
+    <origin xyz="-0.184088 0.022403 -0.1615" rpy="0 0 0"/>
     <geometry>
       <mesh filename="package://cube_description/meshes/depth_camera_v1_1.stl" scale="0.001 0.001 0.001"/>
@@ -77,90 +90,70 @@
   </collision>
 </link>
-<link name="lidar_v1_1">
+<link name="left_wheel_v1_1">
   <inertial>
-    <origin xyz="7.385233546074017e-18 0.0 0.010000000000000009" rpy="0 0 0"/>
-    <mass value="0.6042068071016569"/>
-    <inertia ixx="0.000205" iyy="0.000205" izz="0.00037" ixy="0.0" iyz="0.0" ixz="0.0"/>
+    <origin xyz="-0.00011476068027998013 0.057486019860003096 1.811551186836624e-10" rpy="0 0 0"/>
+    <mass value="4.364871932625406"/>
+    <inertia ixx="0.007848" iyy="0.014009" izz="0.007848" ixy="-1.2e-05" iyz="-0.0" ixz="0.0"/>
   </inertial>
   <visual>
-    <origin xyz="-0.0 -0.0 -0.1755" rpy="0 0 0"/>
+    <origin xyz="0.014189 -0.115701 -0.08" rpy="0 0 0"/>
     <geometry>
-      <mesh filename="package://cube_description/meshes/lidar_v1_1.stl" scale="0.001 0.001 0.001"/>
+      <mesh filename="package://cube_description/meshes/left_wheel_v1_1.stl" scale="0.001 0.001 0.001"/>
     </geometry>
     <material name="steel_satin"/>
   </visual>
   <collision>
-    <origin xyz="-0.0 -0.0 -0.1755" rpy="0 0 0"/>
+    <origin xyz="0.014189 -0.115701 -0.08" rpy="0 0 0"/>
     <geometry>
-      <mesh filename="package://cube_description/meshes/lidar_v1_1.stl" scale="0.001 0.001 0.001"/>
+      <mesh filename="package://cube_description/meshes/left_wheel_v1_1.stl" scale="0.001 0.001 0.001"/>
     </geometry>
   </collision>
 </link>
-<link name="right_wheel_v3_1">
+<link name="right_wheel_v1_1">
   <inertial>
-    <origin xyz="1.269686219929395e-17 -0.020000000000000018 0.0" rpy="0 0 0"/>
-    <mass value="5.623069146418319"/>
-    <inertia ixx="0.008763" iyy="0.016026" izz="0.008763" ixy="0.0" iyz="0.0" ixz="-0.0"/>
+    <origin xyz="0.00011493441134234963 -0.05748636841054998 -1.8113159583332816e-10" rpy="0 0 0"/>
+    <mass value="4.364871932625406"/>
+    <inertia ixx="0.007848" iyy="0.014009" izz="0.007848" ixy="-1.2e-05" iyz="-0.0" ixz="0.0"/>
   </inertial>
   <visual>
-    <origin xyz="-0.0 0.205 -0.0755" rpy="0 0 0"/>
+    <origin xyz="0.013725 0.116298 -0.08" rpy="0 0 0"/>
     <geometry>
-      <mesh filename="package://cube_description/meshes/right_wheel_v3_1.stl" scale="0.001 0.001 0.001"/>
+      <mesh filename="package://cube_description/meshes/right_wheel_v1_1.stl" scale="0.001 0.001 0.001"/>
     </geometry>
     <material name="steel_satin"/>
   </visual>
   <collision>
-    <origin xyz="-0.0 0.205 -0.0755" rpy="0 0 0"/>
+    <origin xyz="0.013725 0.116298 -0.08" rpy="0 0 0"/>
     <geometry>
-      <mesh filename="package://cube_description/meshes/right_wheel_v3_1.stl" scale="0.001 0.001 0.001"/>
-    </geometry>
-  </collision>
-</link>
-<link name="left_wheel_v3_1">
-  <inertial>
-    <origin xyz="1.269686219929395e-17 0.020000000000000018 0.0" rpy="0 0 0"/>
-    <mass value="5.623069146418319"/>
-    <inertia ixx="0.008763" iyy="0.016026" izz="0.008763" ixy="-0.0" iyz="0.0" ixz="-0.0"/>
-  </inertial>
-  <visual>
-    <origin xyz="-0.0 -0.205 -0.0755" rpy="0 0 0"/>
-    <geometry>
-      <mesh filename="package://cube_description/meshes/left_wheel_v3_1.stl" scale="0.001 0.001 0.001"/>
-    </geometry>
-    <material name="steel_satin"/>
-  </visual>
-  <collision>
-    <origin xyz="-0.0 -0.205 -0.0755" rpy="0 0 0"/>
-    <geometry>
-      <mesh filename="package://cube_description/meshes/left_wheel_v3_1.stl" scale="0.001 0.001 0.001"/>
+      <mesh filename="package://cube_description/meshes/right_wheel_v1_1.stl" scale="0.001 0.001 0.001"/>
     </geometry>
   </collision>
 </link>
 <joint name="Rigid 1" type="fixed">
-  <origin xyz="-0.1 0.0 0.1055" rpy="0 0 0"/>
+  <origin xyz="-0.052922 -0.082837 0.2515" rpy="0 0 0"/>
   <parent link="base_link"/>
   <child link="imu_v1_1"/>
 </joint>
+<joint name="Rigid 2" type="fixed">
+  <origin xyz="0.128043 -1.5e-05 0.1955" rpy="0 0 0"/>
+  <parent link="base_link"/>
+  <child link="lidar_v1_1"/>
+</joint>
 <joint name="Rigid 3" type="fixed">
-  <origin xyz="0.28 0.0 0.0805" rpy="0 0 0"/>
+  <origin xyz="0.184088 -0.022403 0.1615" rpy="0 0 0"/>
   <parent link="base_link"/>
   <child link="depth_camera_v1_1"/>
 </joint>
-<joint name="Rigid 6" type="fixed">
-  <origin xyz="0.0 0.0 0.1755" rpy="0 0 0"/>
+<joint name="Revolute 4" type="continuous">
+  <origin xyz="-0.014189 0.12 0.08" rpy="0 0 0"/>
   <parent link="base_link"/>
-  <child link="lidar_v1_1"/>
+  <child link="left_wheel_v1_1"/>
+  <axis xyz="-0.001999 0.999998 0.0"/>
 </joint>
-<joint name="Revolute 9" type="continuous">
-  <origin xyz="0.0 -0.205 0.0755" rpy="0 0 0"/>
-  <parent link="base_footprint"/>
-  <child link="right_wheel_v3_1"/>
-  <axis xyz="0.0 1.0 0.0"/>
-</joint>
-<joint name="Revolute 10" type="continuous">
-  <origin xyz="0.0 0.205 0.0755" rpy="0 0 0"/>
-  <parent link="base_footprint"/>
-  <child link="left_wheel_v3_1"/>
-  <axis xyz="0.0 1.0 0.0"/>
+<joint name="Revolute 5" type="continuous">
+  <origin xyz="-0.013725 -0.12 0.08" rpy="0 0 0"/>
+  <parent link="base_link"/>
+  <child link="right_wheel_v1_1"/>
+  <axis xyz="0.001999 0.999998 -0.0"/>
 </joint>
 </robot>

File: ros2/src/cube_description/urdf/gazebo.xacro (robot description, xacro)
@@ -28,5 +28,5 @@
     <selfCollide>true</selfCollide>
   </gazebo>
-  <gazebo reference="left_wheel_v3_1">
+  <gazebo reference="left_wheel_v1_1">
     <material>${body_color}</material>
     <mu1>1000</mu1>
@@ -34,5 +34,5 @@
     <selfCollide>true</selfCollide>
   </gazebo>
-  <gazebo reference="right_wheel_v3_1">
+  <gazebo reference="right_wheel_v1_1">
     <material>${body_color}</material>
     <mu1>1000</mu1>
@@ -45,9 +45,9 @@
       <update_rate>50</update_rate>
       <!-- wheels -->
-      <left_joint>Revolute 10</left_joint>
-      <right_joint>Revolute 9</right_joint>
+      <left_joint>Revolute 4</left_joint>
+      <right_joint>Revolute 5</right_joint>
       <!-- kinematics -->
-      <wheel_separation>0.45</wheel_separation>
-      <wheel_diameter>0.15</wheel_diameter>
+      <wheel_separation>0.344</wheel_separation>
+      <wheel_diameter>0.16</wheel_diameter>
       <!-- input -->
       <command_topic>cmd_vel</command_topic>

File: ros2/src/cube_description/urdf/materials.xacro (robot description, xacro)
@@ -4,6 +4,12 @@
   <color rgba="0.700 0.700 0.700 1.000"/>
 </material>
+<material name="opaque160160160">
+  <color rgba="0.6274509803921569 0.6274509803921569 0.6274509803921569 1.0"/>
+</material>
 <material name="steel_satin">
   <color rgba="0.6274509803921569 0.6274509803921569 0.6274509803921569 1.0"/>
 </material>
+<material name="opaque262626">
+  <color rgba="0.10196078431372549 0.10196078431372549 0.10196078431372549 1.0"/>
+</material>
 </robot>

Commit message: changed urdf and composefile

File: ros2/src/cube_description/urdf/cube.xacro (robot description, xacro)
@@ -9,4 +9,6 @@
   <parent link="base_footprint" />
   <child link="base_link" />
+  <origin xyz="0 0 0" rpy="0 0 0"/>
+  <axis xyz="0 0 0"/>
 </joint>
 <link name="base_link">
@@ -17,5 +19,5 @@
   </inertial>
   <visual>
-    <origin xyz="0 0 0" rpy="0 0 0"/>
+    <origin xyz="0 0 0.0" rpy="0 0 0"/>
     <geometry>
       <mesh filename="package://cube_description/meshes/base_link.stl" scale="0.001 0.001 0.001"/>
@@ -24,7 +26,8 @@
   </visual>
   <collision>
-    <origin xyz="0 0 0" rpy="0 0 0"/>
+    <origin xyz="0 0 0.006" rpy="0 0 0"/>
     <geometry>
-      <mesh filename="package://cube_description/meshes/base_link.stl" scale="0.001 0.001 0.001"/>
+      <!-- <mesh filename="package://cube_description/meshes/base_link.stl" scale="0.001 0.001 0.001"/> -->
+      <box size="0.45 0.05 0.01" />
     </geometry>
   </collision>
@@ -149,5 +152,5 @@
   <parent link="base_link"/>
   <child link="left_wheel_v1_1"/>
-  <axis xyz="-0.001999 0.999998 0.0"/>
+  <axis xyz="-0.0 1.0 0.0"/>
 </joint>
 <joint name="Revolute 5" type="continuous">
@@ -155,5 +158,5 @@
   <parent link="base_link"/>
   <child link="right_wheel_v1_1"/>
-  <axis xyz="0.001999 0.999998 -0.0"/>
+  <axis xyz="0.0 1.0 -0.0"/>
 </joint>
 </robot>

File: ros2/src/cube_description/urdf/gazebo.xacro (robot description, xacro)
@@ -5,6 +5,6 @@
   <gazebo reference="base_link">
     <material>${body_color}</material>
-    <mu1>0.2</mu1>
-    <mu2>0.2</mu2>
+    <mu1>0.1</mu1>
+    <mu2>0.1</mu2>
     <selfCollide>true</selfCollide>
     <gravity>true</gravity>
